File: EUROSCART_2_JP21.sch (KiCad schematic (older format))
At the start: 2 parts, among them J1 SCART-F, J2 SCART-F

Commit message: revised to use one female and one male
Parts:
- J1: footprint SCART-RIGHT-ANGLE:SCART Right Angle -> Tinkerplunk:MALE_SCART; symbol SCART-F -> EUROSCART_2_JP21-rescue:SCART-F
- J2: footprint SCART-RIGHT-ANGLE:SCART Right Angle -> Tinkerplunk:SCART-F-RA; symbol SCART-F -> EUROSCART_2_JP21-rescue:SCART-F
Changed lines of the file:
@@
-EESchema Schematic File Version 2
-LIBS:power
-LIBS:device
-LIBS:switches
-LIBS:relays
-LIBS:motors
-LIBS:transistors
-LIBS:conn
-LIBS:linear
-LIBS:regul
-LIBS:74xx
-LIBS:cmos4000
-LIBS:adc-dac
-LIBS:memory
-LIBS:xilinx
-LIBS:microcontrollers
-LIBS:dsp
-LIBS:microchip
-LIBS:analog_switches
-LIBS:motorola
-LIBS:texas
-LIBS:intel
-LIBS:audio
-LIBS:interface
-LIBS:digital-audio
-LIBS:philips
-LIBS:display
-LIBS:cypress
-LIBS:siliconi
-LIBS:opto
-LIBS:atmel
-LIBS:contrib
-LIBS:valves
-EELAYER 25 0
+EESchema Schematic File Version 4
+LIBS:EUROSCART_2_JP21-cache
+EELAYER 29 0
 EELAYER END
 $Descr A4 11693 8268
@@
 $EndDescr
 $Comp
-L SCART-F J1
+L EUROSCART_2_JP21-rescue:SCART-F J1
 U 1 1 5B540E82
 P 3625 3375
 F 0 "J1" H 3625 4575 50  0000 C CNN
 F 1 "SCART-F" H 3665 2175 50  0000 C CNN
-F 2 "SCART-RIGHT-ANGLE:SCART Right Angle" H 3625 3375 50  0001 C CNN
+F 2 "Tinkerplunk:MALE_SCART" H 3625 3375 50  0001 C CNN
 F 3 "" H 3625 3375 50  0001 C CNN
 	1    3625 3375
@@
 $EndComp
 $Comp
-L SCART-F J2
+L EUROSCART_2_JP21-rescue:SCART-F J2
 U 1 1 5B540EA9
 P 5800 3375
 F 0 "J2" H 5800 4575 50  0000 C CNN
 F 1 "SCART-F" H 5840 2175 50  0000 C CNN
-F 2 "SCART-RIGHT-ANGLE:SCART Right Angle" H 5800 3375 50  0001 C CNN
+F 2 "Tinkerplunk:SCART-F-RA" H 5800 3375 50  0001 C CNN
 F 3 "" H 5800 3375 50  0001 C CNN
 	1    5800 3375

Commit message: Fixed swapped sync pins on JP21
Connections:
- net S_IN: now also J2.9 (P9); no longer J2.10 (P10)
- net S_OUT: now also J2.10 (P10); no longer J2.9 (P9)
Changed lines of the file:
@@
 Text GLabel 4225 2525 2    60   Input ~ 0
 S_IN
-Text GLabel 6400 3525 2    60   Input ~ 0
-S_IN
 Text GLabel 3025 2625 0    60   Input ~ 0
-S_OUT
-Text GLabel 5200 3625 0    60   Input ~ 0
 S_OUT
 Text GLabel 3025 3025 0    60   Input ~ 0
@@
 NoConn ~ 4225 3325
 NoConn ~ 4225 3525
+Text GLabel 5200 3625 0    60   Input ~ 0
+S_IN
+Text GLabel 6400 3525 2    60   Input ~ 0
+S_OUT
 $EndSCHEMATC
