File: JP21F_to_EUROM.sch (KiCad schematic (older format))
At the start: 2 parts, among them J1 SCART-F, J2 SCART-F

Commit message: fixed incorrect audio pins for JP21
Parts:
- J1, J2: symbol EUROSCART_2_JP21-rescue:SCART-F -> JP21F_to_EUROM-rescue:SCART-F-EUROSCART_2_JP21-rescue
Connections:
- net L_IN: now also J2.1 (P1); no longer J2.2 (P2)
- net L_OUT: now also J2.2 (P2); no longer J2.1 (P1)
- net RT_IN: now also J2.5 (P5); no longer J2.6 (P6)
- net RT_OUT: now also J2.6 (P6); no longer J2.5 (P5)
Changed lines of the file:
@@
 EESchema Schematic File Version 4
-LIBS:EUROSCART_2_JP21-cache
+LIBS:JP21F_to_EUROM-cache
 EELAYER 29 0
 EELAYER END
@@
 $EndDescr
 $Comp
-L EUROSCART_2_JP21-rescue:SCART-F J1
+L JP21F_to_EUROM-rescue:SCART-F-EUROSCART_2_JP21-rescue J1
 U 1 1 5B540E82
 P 3625 3375
@@
 $EndComp
 $Comp
-L EUROSCART_2_JP21-rescue:SCART-F J2
+L JP21F_to_EUROM-rescue:SCART-F-EUROSCART_2_JP21-rescue J2
 U 1 1 5B540EA9
 P 5800 3375
@@
 RT_OUT
 Text GLabel 5200 4025 0    60   Input ~ 0
-RT_OUT
+RT_IN
 Text GLabel 4225 4125 2    60   Input ~ 0
 A_GND
@@
 RT_IN
 Text GLabel 6400 3925 2    60   Input ~ 0
-RT_IN
+RT_OUT
 Text GLabel 3025 4225 0    60   Input ~ 0
 L_OUT
 Text GLabel 5200 4425 0    60   Input ~ 0
-L_OUT
+L_IN
 Text GLabel 4225 3925 2    60   Input ~ 0
 L_IN
 Text GLabel 6400 4325 2    60   Input ~ 0
-L_IN
+L_OUT
 Text GLabel 4225 2525 2    60   Input ~ 0
 S_IN
